File: 808_output.sch (EAGLE design)
At the start: 31 parts, among them IC1 TL072P

Commit message: layout
Parts:
- BD, CB, CH, CP, CY, HT, LT, MT, OH, RS, SD: device rcl:R-US_0207/7 -> rcl:R-US_0207/5V
- OUTPUT: value AUDIO-JACK -> 22-23-2021; device erthenvar:AUDIO-JACK -> con-molex:22-23-2021
Connections:
- removed net N$24: C8.2, D1.A, D2.C, IC1B.OUT, OUTPUT.TIP, R3.2
- new net N$19: C8.2, D1.A, D2.C, IC1B.OUT, OUTPUT-2.S, R3.2
- net N$26: now also OUTPUT-1.S; no longer OUTPUT.RING
Changed lines of the file:
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@@
 </variantdefs>
 <classes>
-<class number="0" name="default" width="0" drill="0">
+<class number="0" name="default" width="0.635" drill="0.254">
+<clearance class="0" value="0.254"/>
+</class>
+<class number="1" name="GND" width="1.016" drill="1.016">
+<clearance class="1" value="0.508"/>
 </class>
 </classes>
@@
 <part name="C4" library="rcl" deviceset="C-US" device="050-024X044" value="100n"/>
 <part name="C5" library="rcl" deviceset="C-US" device="050-024X044" value="100n"/>
-<part name="BD" library="rcl" deviceset="R-US_" device="0207/7" value="22k"/>
-<part name="SD" library="rcl" deviceset="R-US_" device="0207/7" value="33k"/>
-<part name="LT" library="rcl" deviceset="R-US_" device="0207/7" value="33k"/>
-<part name="MT" library="rcl" deviceset="R-US_" device="0207/7" value="33k"/>
-<part name="HT" library="rcl" deviceset="R-US_" device="0207/7" value="33k"/>
-<part name="RS" library="rcl" deviceset="R-US_" device="0207/7" value="33k"/>
-<part name="CP" library="rcl" deviceset="R-US_" device="0207/7" value="33k"/>
-<part name="OH" library="rcl" deviceset="R-US_" device="0207/7" value="56k"/>
-<part name="CH" library="rcl" deviceset="R-US_" device="0207/7" value="47k"/>
-<part name="CB" library="rcl" deviceset="R-US_" device="0207/7" value="47k"/>
-<part name="CY" library="rcl" deviceset="R-US_" device="0207/7" value="47k"/>
+<part name="BD" library="rcl" deviceset="R-US_" device="0207/5V" value="22k"/>
+<part name="SD" library="rcl" deviceset="R-US_" device="0207/5V" value="33k"/>
+<part name="LT" library="rcl" deviceset="R-US_" device="0207/5V" value="33k"/>
+<part name="MT" library="rcl" deviceset="R-US_" device="0207/5V" value="33k"/>
+<part name="HT" library="rcl" deviceset="R-US_" device="0207/5V" value="33k"/>
+<part name="RS" library="rcl" deviceset="R-US_" device="0207/5V" value="33k"/>
+<part name="CP" library="rcl" deviceset="R-US_" device="0207/5V" value="33k"/>
+<part name="OH" library="rcl" deviceset="R-US_" device="0207/5V" value="56k"/>
+<part name="CH" library="rcl" deviceset="R-US_" device="0207/5V" value="47k"/>
+<part name="CB" library="rcl" deviceset="R-US_" device="0207/5V" value="47k"/>
+<part name="CY" library="rcl" deviceset="R-US_" device="0207/5V" value="47k"/>
 <part name="X1" library="con-molex" deviceset="KK-156-11" device=""/>
 <part name="IC1" library="linear" deviceset="TL072" device="P"/>
@@
 <part name="P-2" library="supply1" deviceset="-12V" device=""/>
 <part name="GND2" library="supply1" deviceset="GND" device=""/>
-<part name="OUTPUT" library="erthenvar" deviceset="AUDIO-JACK" device=""/>
 <part name="GND4" library="supply1" deviceset="GND" device=""/>
 <part name="R1" library="rcl" deviceset="R-US_" device="0207/7" value="33k"/>
@@
 <part name="P+3" library="supply1" deviceset="+12V" device=""/>
 <part name="P-3" library="supply1" deviceset="-12V" device=""/>
+<part name="OUTPUT" library="con-molex" deviceset="22-23-2021" device=""/>
 </parts>
 <sheets>
@@
 <instance part="P-2" gate="1" x="139.7" y="7.62"/>
 <instance part="GND2" gate="1" x="157.48" y="20.32"/>
-<instance part="OUTPUT" gate="G$1" x="154.94" y="60.96" rot="R180"/>
-<instance part="GND4" gate="1" x="147.32" y="53.34"/>
+<instance part="GND4" gate="1" x="149.86" y="53.34"/>
 <instance part="R1" gate="G$1" x="86.36" y="83.82"/>
 <instance part="R2" gate="G$1" x="104.14" y="68.58"/>
@@
 <instance part="P+3" gate="1" x="142.24" y="81.28"/>
 <instance part="P-3" gate="1" x="142.24" y="50.8"/>
+<instance part="OUTPUT" gate="-1" x="154.94" y="63.5" rot="MR180"/>
+<instance part="OUTPUT" gate="-2" x="154.94" y="66.04" rot="MR180"/>
 </instances>
 <busses>
@@
 </segment>
 <segment>
-<pinref part="OUTPUT" gate="G$1" pin="RING"/>
 <pinref part="GND4" gate="1" pin="GND"/>
-<wire x1="147.32" y1="55.88" x2="147.32" y2="58.42" width="0.1524" layer="91"/>
+<pinref part="OUTPUT" gate="-1" pin="S"/>
+<wire x1="152.4" y1="63.5" x2="149.86" y2="63.5" width="0.1524" layer="91"/>
+<wire x1="149.86" y1="63.5" x2="149.86" y2="55.88" width="0.1524" layer="91"/>
 </segment>
 </net>
@@
 </segment>
 </net>
-<net name="N$24" class="0">
-<segment>
-<pinref part="OUTPUT" gate="G$1" pin="TIP"/>
-<wire x1="147.32" y1="66.04" x2="142.24" y2="66.04" width="0.1524" layer="91"/>
+<net name="N$15" class="0">
+<segment>
+<pinref part="R2" gate="G$1" pin="1"/>
+<pinref part="IC1" gate="A" pin="OUT"/>
+<wire x1="93.98" y1="68.58" x2="96.52" y2="68.58" width="0.1524" layer="91"/>
+<pinref part="C7" gate="G$1" pin="2"/>
+<wire x1="96.52" y1="68.58" x2="99.06" y2="68.58" width="0.1524" layer="91"/>
+<wire x1="88.9" y1="88.9" x2="96.52" y2="88.9" width="0.1524" layer="91"/>
+<wire x1="96.52" y1="88.9" x2="96.52" y2="83.82" width="0.1524" layer="91"/>
+<junction x="96.52" y="68.58"/>
+<pinref part="R1" gate="G$1" pin="2"/>
+<wire x1="96.52" y1="83.82" x2="96.52" y2="68.58" width="0.1524" layer="91"/>
+<wire x1="91.44" y1="83.82" x2="96.52" y2="83.82" width="0.1524" layer="91"/>
+<junction x="96.52" y="83.82"/>
+</segment>
+</net>
+<net name="N$16" class="0">
+<segment>
+<pinref part="IC1" gate="B" pin="-IN"/>
+<pinref part="R2" gate="G$1" pin="2"/>
+<wire x1="109.22" y1="68.58" x2="111.76" y2="68.58" width="0.1524" layer="91"/>
+<pinref part="C8" gate="G$1" pin="1"/>
+<wire x1="111.76" y1="68.58" x2="114.3" y2="68.58" width="0.1524" layer="91"/>
+<wire x1="116.84" y1="83.82" x2="111.76" y2="83.82" width="0.1524" layer="91"/>
+<wire x1="111.76" y1="83.82" x2="111.76" y2="78.74" width="0.1524" layer="91"/>
+<junction x="111.76" y="68.58"/>
+<pinref part="R3" gate="G$1" pin="1"/>
+<wire x1="111.76" y1="78.74" x2="111.76" y2="68.58" width="0.1524" layer="91"/>
+<wire x1="116.84" y1="78.74" x2="111.76" y2="78.74" width="0.1524" layer="91"/>
+<junction x="111.76" y="78.74"/>
+</segment>
+</net>
+<net name="N$17" class="0">
+<segment>
+<pinref part="IC1" gate="A" pin="-IN"/>
+<wire x1="78.74" y1="71.12" x2="76.2" y2="71.12" width="0.1524" layer="91"/>
+<pinref part="C7" gate="G$1" pin="1"/>
+<wire x1="81.28" y1="88.9" x2="76.2" y2="88.9" width="0.1524" layer="91"/>
+<wire x1="76.2" y1="88.9" x2="76.2" y2="83.82" width="0.1524" layer="91"/>
+<pinref part="R1" gate="G$1" pin="1"/>
+<wire x1="81.28" y1="83.82" x2="76.2" y2="83.82" width="0.1524" layer="91"/>
+<junction x="76.2" y="83.82"/>
+<wire x1="76.2" y1="83.82" x2="76.2" y2="71.12" width="0.1524" layer="91"/>
+<pinref part="C9" gate="G$1" pin="-"/>
+<wire x1="71.12" y1="71.12" x2="76.2" y2="71.12" width="0.1524" layer="91"/>
+<junction x="76.2" y="71.12"/>
+</segment>
+</net>
+<net name="N$19" class="0">
+<segment>
+<pinref part="OUTPUT" gate="-2" pin="S"/>
+<wire x1="152.4" y1="66.04" x2="142.24" y2="66.04" width="0.1524" layer="91"/>
 <pinref part="C8" gate="G$1" pin="2"/>
 <wire x1="142.24" y1="66.04" x2="132.08" y2="66.04" width="0.1524" layer="91"/>
@@
 </segment>
 </net>
-<net name="N$15" class="0">
-<segment>
-<pinref part="R2" gate="G$1" pin="1"/>
-<pinref part="IC1" gate="A" pin="OUT"/>
-<wire x1="93.98" y1="68.58" x2="96.52" y2="68.58" width="0.1524" layer="91"/>
-<pinref part="C7" gate="G$1" pin="2"/>
-<wire x1="96.52" y1="68.58" x2="99.06" y2="68.58" width="0.1524" layer="91"/>
-<wire x1="88.9" y1="88.9" x2="96.52" y2="88.9" width="0.1524" layer="91"/>
-<wire x1="96.52" y1="88.9" x2="96.52" y2="83.82" width="0.1524" layer="91"/>
-<junction x="96.52" y="68.58"/>
-<pinref part="R1" gate="G$1" pin="2"/>
-<wire x1="96.52" y1="83.82" x2="96.52" y2="68.58" width="0.1524" layer="91"/>
-<wire x1="91.44" y1="83.82" x2="96.52" y2="83.82" width="0.1524" layer="91"/>
-<junction x="96.52" y="83.82"/>
-</segment>
-</net>
-<net name="N$16" class="0">
-<segment>
-<pinref part="IC1" gate="B" pin="-IN"/>
-<pinref part="R2" gate="G$1" pin="2"/>
-<wire x1="109.22" y1="68.58" x2="111.76" y2="68.58" width="0.1524" layer="91"/>
-<pinref part="C8" gate="G$1" pin="1"/>
-<wire x1="111.76" y1="68.58" x2="114.3" y2="68.58" width="0.1524" layer="91"/>
-<wire x1="116.84" y1="83.82" x2="111.76" y2="83.82" width="0.1524" layer="91"/>
-<wire x1="111.76" y1="83.82" x2="111.76" y2="78.74" width="0.1524" layer="91"/>
-<junction x="111.76" y="68.58"/>
-<pinref part="R3" gate="G$1" pin="1"/>
-<wire x1="111.76" y1="78.74" x2="111.76" y2="68.58" width="0.1524" layer="91"/>
-<wire x1="116.84" y1="78.74" x2="111.76" y2="78.74" width="0.1524" layer="91"/>
-<junction x="111.76" y="78.74"/>
-</segment>
-</net>
-<net name="N$17" class="0">
-<segment>
-<pinref part="IC1" gate="A" pin="-IN"/>
-<wire x1="78.74" y1="71.12" x2="76.2" y2="71.12" width="0.1524" layer="91"/>
-<pinref part="C7" gate="G$1" pin="1"/>
-<wire x1="81.28" y1="88.9" x2="76.2" y2="88.9" width="0.1524" layer="91"/>
-<wire x1="76.2" y1="88.9" x2="76.2" y2="83.82" width="0.1524" layer="91"/>
-<pinref part="R1" gate="G$1" pin="1"/>
-<wire x1="81.28" y1="83.82" x2="76.2" y2="83.82" width="0.1524" layer="91"/>
-<junction x="76.2" y="83.82"/>
-<wire x1="76.2" y1="83.82" x2="76.2" y2="71.12" width="0.1524" layer="91"/>
-<pinref part="C9" gate="G$1" pin="-"/>
-<wire x1="71.12" y1="71.12" x2="76.2" y2="71.12" width="0.1524" layer="91"/>
-<junction x="76.2" y="71.12"/>
-</segment>
-</net>

Commit message: closer to og 808
Parts:
- added C10, C11: 1uF/50v, rcl:CPOL-USB45181A
- added C12: 10uF Bi, rcl:CPOL-USB45181A
- added VOLUME_POT: (no value), con-molex:KK-156-3
- C9: device rcl:CPOL-USB45181A -> rcl:CPOL-USB45181B
Connections:
- new net N$18: C11.-, R2.1
- new net N$20: C10.+, VOLUME_POT-3.S
- new net N$21: C11.+, VOLUME_POT-2.S
- new net N$22: C12.-, OUTPUT-2.S
- net GND: now also VOLUME_POT-1.S
- net N$15: now also C10.-; no longer R2.1
- net N$19: now also C12.+; no longer OUTPUT-2.S
Other:
- moved on the sheet: BD, C1, C2, C3, C4, C5, C6, C8, C9, CB, CH, CP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

Commit message: routed
Parts:
- C9: device rcl:CPOL-USB45181B -> rcl:CPOL-USB45181A
Connections:
- removed net N$26: C1.-, C2.+, C4.2, C5.1, OUTPUT-1.S, PWR1.GND
- net GND: now also C1.-, C2.+, C4.2, C5.1, OUTPUT-1.S, PWR1.GND
Changed lines of the file:
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@@
 <part name="P+1" library="supply1" deviceset="+12V" device=""/>
 <part name="P-1" library="supply1" deviceset="-12V" device=""/>
-<part name="GND1" library="supply1" deviceset="GND" device=""/>
 <part name="C4" library="rcl" deviceset="C-US" device="050-024X044" value="100n"/>
 <part name="C5" library="rcl" deviceset="C-US" device="050-024X044" value="100n"/>
@@
 <part name="P+2" library="supply1" deviceset="+12V" device=""/>
 <part name="P-2" library="supply1" deviceset="-12V" device=""/>
-<part name="GND2" library="supply1" deviceset="GND" device=""/>
-<part name="GND4" library="supply1" deviceset="GND" device=""/>
 <part name="R1" library="rcl" deviceset="R-US_" device="0207/7" value="33k"/>
 <part name="R2" library="rcl" deviceset="R-US_" device="0207/7" value="22k"/>
@@
 <part name="C7" library="rcl" deviceset="C-US" device="025-025X050" value="220p"/>
 <part name="C8" library="rcl" deviceset="C-US" device="025-025X050" value="220p"/>
-<part name="GND3" library="supply1" deviceset="GND" device=""/>
-<part name="GND5" library="supply1" deviceset="GND" device=""/>
-<part name="C9" library="rcl" deviceset="CPOL-US" device="B45181B" value="1uF/50v"/>
+<part name="C9" library="rcl" deviceset="CPOL-US" device="B45181A" value="1uF/50v"/>
 <part name="D1" library="808_lt" deviceset="DIODE" device="DO-1N4148"/>
 <part name="D2" library="808_lt" deviceset="DIODE" device="DO-1N4148"/>
@@
 <part name="C11" library="rcl" deviceset="CPOL-US" device="B45181A" value="1uF/50v"/>
 <part name="VOLUME_POT" library="con-molex" deviceset="KK-156-3" device=""/>
+<part name="C12" library="rcl" deviceset="CPOL-US" device="B45181A" value="10uF Bi"/>
+<part name="GND1" library="supply1" deviceset="GND" device=""/>
+<part name="GND2" library="supply1" deviceset="GND" device=""/>
+<part name="GND3" library="supply1" deviceset="GND" device=""/>
+<part name="GND4" library="supply1" deviceset="GND" device=""/>
+<part name="GND5" library="supply1" deviceset="GND" device=""/>
 <part name="GND6" library="supply1" deviceset="GND" device=""/>
-<part name="C12" library="rcl" deviceset="CPOL-US" device="B45181A" value="10uF Bi"/>
 </parts>
 <sheets>
@@
 <instance part="P+1" gate="1" x="127" y="40.64"/>
 <instance part="P-1" gate="1" x="127" y="5.08"/>
-<instance part="GND1" gate="1" x="144.78" y="17.78"/>
 <instance part="C4" gate="G$1" x="134.62" y="30.48"/>
 <instance part="C5" gate="G$1" x="134.62" y="17.78"/>
@@
 <instance part="P+2" gate="1" x="157.48" y="40.64"/>
 <instance part="P-2" gate="1" x="157.48" y="5.08"/>
-<instance part="GND2" gate="1" x="175.26" y="17.78"/>
-<instance part="GND4" gate="1" x="190.5" y="53.34"/>
 <instance part="R1" gate="G$1" x="86.36" y="83.82"/>
 <instance part="R2" gate="G$1" x="132.08" y="68.58"/>
@@
 <instance part="C7" gate="G$1" x="83.82" y="88.9" rot="R90"/>
 <instance part="C8" gate="G$1" x="147.32" y="83.82" rot="R90"/>
-<instance part="GND3" gate="1" x="142.24" y="58.42"/>
-<instance part="GND5" gate="1" x="78.74" y="58.42"/>
 <instance part="C9" gate="G$1" x="68.58" y="71.12" rot="R90"/>
 <instance part="D1" gate="G$1" x="170.18" y="73.66" rot="R90"/>
@@
 <instance part="VOLUME_POT" gate="-2" x="104.14" y="53.34" rot="R180"/>
 <instance part="VOLUME_POT" gate="-3" x="104.14" y="55.88" rot="R180"/>
-<instance part="GND6" gate="1" x="106.68" y="48.26"/>
 <instance part="C12" gate="G$1" x="180.34" y="66.04" rot="R90"/>
+<instance part="GND1" gate="1" x="78.74" y="58.42"/>
+<instance part="GND2" gate="1" x="109.22" y="45.72"/>
+<instance part="GND3" gate="1" x="142.24" y="58.42"/>
+<instance part="GND4" gate="1" x="190.5" y="53.34"/>
+<instance part="GND5" gate="1" x="175.26" y="17.78"/>
+<instance part="GND6" gate="1" x="144.78" y="17.78"/>
 </instances>
 <busses>
@@
 <pinref part="P-3" gate="1" pin="-12V"/>
 <wire x1="170.18" y1="53.34" x2="170.18" y2="55.88" width="0.1524" layer="91"/>
-</segment>
-</net>
-<net name="N$26" class="0">
-<segment>
-<pinref part="PWR1" gate="G$1" pin="GND"/>
-<pinref part="GND1" gate="1" pin="GND"/>
-<wire x1="104.14" y1="22.86" x2="127" y2="22.86" width="0.1524" layer="91"/>
-<wire x1="127" y1="22.86" x2="134.62" y2="22.86" width="0.1524" layer="91"/>
-<wire x1="134.62" y1="22.86" x2="144.78" y2="22.86" width="0.1524" layer="91"/>
-<wire x1="144.78" y1="22.86" x2="144.78" y2="20.32" width="0.1524" layer="91"/>
-<pinref part="C1" gate="G$1" pin="-"/>
-<wire x1="127" y1="25.4" x2="127" y2="22.86" width="0.1524" layer="91"/>
-<junction x="127" y="22.86"/>
-<pinref part="C2" gate="G$1" pin="+"/>
-<wire x1="127" y1="20.32" x2="127" y2="22.86" width="0.1524" layer="91"/>
-<pinref part="C4" gate="G$1" pin="2"/>
-<wire x1="134.62" y1="25.4" x2="134.62" y2="22.86" width="0.1524" layer="91"/>
-<junction x="134.62" y="22.86"/>
-<pinref part="C5" gate="G$1" pin="1"/>
-<wire x1="134.62" y1="20.32" x2="134.62" y2="22.86" width="0.1524" layer="91"/>
-</segment>
-<segment>
-<pinref part="GND4" gate="1" pin="GND"/>
-<pinref part="OUTPUT" gate="-1" pin="S"/>
-<wire x1="193.04" y1="63.5" x2="190.5" y2="63.5" width="0.1524" layer="91"/>
-<wire x1="190.5" y1="63.5" x2="190.5" y2="55.88" width="0.1524" layer="91"/>
-</segment>
-</net>
-<net name="GND" class="0">
-<segment>
-<pinref part="C3" gate="G$1" pin="2"/>
-<wire x1="167.64" y1="25.4" x2="167.64" y2="22.86" width="0.1524" layer="91"/>
-<pinref part="C6" gate="G$1" pin="1"/>
-<pinref part="GND2" gate="1" pin="GND"/>
-<wire x1="167.64" y1="22.86" x2="167.64" y2="20.32" width="0.1524" layer="91"/>
-<wire x1="167.64" y1="22.86" x2="175.26" y2="22.86" width="0.1524" layer="91"/>
-<wire x1="175.26" y1="22.86" x2="175.26" y2="20.32" width="0.1524" layer="91"/>
-<junction x="167.64" y="22.86"/>
-</segment>
-<segment>
-<pinref part="IC1" gate="B" pin="+IN"/>
-<pinref part="GND3" gate="1" pin="GND"/>
-<wire x1="142.24" y1="60.96" x2="142.24" y2="63.5" width="0.1524" layer="91"/>
-</segment>
-<segment>
-<pinref part="IC1" gate="A" pin="+IN"/>
-<pinref part="GND5" gate="1" pin="GND"/>
-<wire x1="78.74" y1="60.96" x2="78.74" y2="66.04" width="0.1524" layer="91"/>
-</segment>
-<segment>
-<pinref part="VOLUME_POT" gate="-1" pin="S"/>
-<pinref part="GND6" gate="1" pin="GND"/>
 </segment>
 </net>
@@
 </segment>
 </net>
+<net name="GND" class="0">
+<segment>
+<pinref part="IC1" gate="A" pin="+IN"/>
+<wire x1="78.74" y1="60.96" x2="78.74" y2="66.04" width="0.1524" layer="91"/>
+<pinref part="GND1" gate="1" pin="GND"/>
+</segment>
+<segment>
+<pinref part="VOLUME_POT" gate="-1" pin="S"/>
+<wire x1="106.68" y1="50.8" x2="109.22" y2="50.8" width="0.1524" layer="91"/>
+<wire x1="109.22" y1="50.8" x2="109.22" y2="48.26" width="0.1524" layer="91"/>
+<pinref part="GND2" gate="1" pin="GND"/>
+</segment>
+<segment>
+<pinref part="IC1" gate="B" pin="+IN"/>
+<wire x1="142.24" y1="60.96" x2="142.24" y2="63.5" width="0.1524" layer="91"/>
+<pinref part="GND3" gate="1" pin="GND"/>
+</segment>
+<segment>
+<pinref part="OUTPUT" gate="-1" pin="S"/>
+<wire x1="193.04" y1="63.5" x2="190.5" y2="63.5" width="0.1524" layer="91"/>
+<wire x1="190.5" y1="63.5" x2="190.5" y2="55.88" width="0.1524" layer="91"/>
+<pinref part="GND4" gate="1" pin="GND"/>
+</segment>
+<segment>
+<pinref part="C3" gate="G$1" pin="2"/>
+<wire x1="167.64" y1="25.4" x2="167.64" y2="22.86" width="0.1524" layer="91"/>
+<pinref part="C6" gate="G$1" pin="1"/>
+<wire x1="167.64" y1="22.86" x2="167.64" y2="20.32" width="0.1524" layer="91"/>
+<wire x1="167.64" y1="22.86" x2="175.26" y2="22.86" width="0.1524" layer="91"/>
+<wire x1="175.26" y1="22.86" x2="175.26" y2="20.32" width="0.1524" layer="91"/>
+<junction x="167.64" y="22.86"/>
+<pinref part="GND5" gate="1" pin="GND"/>
+</segment>
+<segment>
+<pinref part="PWR1" gate="G$1" pin="GND"/>
+<wire x1="104.14" y1="22.86" x2="127" y2="22.86" width="0.1524" layer="91"/>
+<wire x1="127" y1="22.86" x2="134.62" y2="22.86" width="0.1524" layer="91"/>
+<wire x1="134.62" y1="22.86" x2="144.78" y2="22.86" width="0.1524" layer="91"/>
+<wire x1="144.78" y1="22.86" x2="144.78" y2="20.32" width="0.1524" layer="91"/>
+<pinref part="C1" gate="G$1" pin="-"/>
+<wire x1="127" y1="25.4" x2="127" y2="22.86" width="0.1524" layer="91"/>
+<junction x="127" y="22.86"/>
+<pinref part="C2" gate="G$1" pin="+"/>
+<wire x1="127" y1="20.32" x2="127" y2="22.86" width="0.1524" layer="91"/>
+<pinref part="C4" gate="G$1" pin="2"/>
+<wire x1="134.62" y1="25.4" x2="134.62" y2="22.86" width="0.1524" layer="91"/>
+<junction x="134.62" y="22.86"/>
+<pinref part="C5" gate="G$1" pin="1"/>
+<wire x1="134.62" y1="20.32" x2="134.62" y2="22.86" width="0.1524" layer="91"/>
+<pinref part="GND6" gate="1" pin="GND"/>
+</segment>
+</net>
